File: Boards/Throttle/throttle.kicad_pcb (KiCad board)
At the start: 2 copper layers, 17 parts, among them U2 TPS561201

Commit message: Worked on layout, finished a VERY rough REV1
Parts:
- added C1: C_0.1uF, footprints:C_0805_OEM, F.Cu at (147.6, 61.0)
- added C10: C_30pF, footprints:C_0805_OEM, F.Cu at (135.0, 77.0)
- added C2: C_0.1uF, footprints:C_0805_OEM, F.Cu at (153.9, 66.5)
- added C4: C_0.1uF, footprints:C_0805_OEM, F.Cu at (134.7, 83.5)
- added C6: C_0.1uF, footprints:C_0805_OEM, F.Cu at (126.3, 71.6)
- added C8: C_100pF, footprints:C_0805_OEM, F.Cu at (129.8, 76.4)
- added C9: C_30pF, footprints:C_0805_OEM, F.Cu at (139.9, 72.5)
- added D10: LED_0805, footprints:LED_0805_OEM, F.Cu at (108.0, 52.1)
- added D3: LED_0805, footprints:LED_0805_OEM, F.Cu at (136.7, 57.9)
- added D4: LED_0805, footprints:LED_0805_OEM, F.Cu at (136.7, 55.1)
- added D5: LED_0805, footprints:LED_0805_OEM, F.Cu at (136.7, 52.3)
- added D6: LED_0805, footprints:LED_0805_OEM, F.Cu at (105.2, 65.8)
- added D8: LED_0805, footprints:LED_0805_OEM, F.Cu at (121.7, 54.2)
- added D9: LED_0805, footprints:LED_0805_OEM, F.Cu at (114.3, 61.0)
- added IC1: ATMEGA16M1, footprints:TQFP-32_7x7mm_Pitch0.8mm, F.Cu at (132.1, 67.2)
- added J1: micromatch_female_TOP_ENTRY_locking_4, footprints:micromatch_female_vert_4, F.Cu at (98.6, 53.3)
- added J2: micromatch_female_TOP_ENTRY_locking_20, footprints:micromatch_female_vert_20, F.Cu at (98.3, 72.0)
- added J3: CONN_02X03, footprints:Pin_Header_Straight_2x03, F.Cu at (151.4, 78.7)
- added Q1: SSM3K333R, footprints:SOT-23F, F.Cu at (109.0, 63.2)
- added Q2: SSM3K333R, footprints:SOT-23F, F.Cu at (124.7, 51.4)
- added Q3: SSM3K333R, footprints:SOT-23F, F.Cu at (117.1, 58.2)
- added Q4: SSM3K333R, footprints:SOT-23F, F.Cu at (111.2, 49.3)
- added R1: R_1M, footprints:R_0805_OEM, F.Cu at (140.3, 63.5)
- added R10: R_200, footprints:R_0805_OEM, F.Cu at (141.7, 55.1)
- added R11: R_200, footprints:R_0805_OEM, F.Cu at (141.7, 52.3)
- added R13: R_1M, footprints:R_0805_OEM, F.Cu at (146.6, 68.8)
- added R14: R_200, footprints:R_0805_OEM, F.Cu at (104.1, 63.2)
- added R15: R_22K, footprints:R_0805_OEM, F.Cu at (99.8, 61.7)
- added R16: R_2.2k, footprints:R_0805_OEM, F.Cu at (150.4, 70.4)
- added R17: R_2.2k, footprints:R_0805_OEM, F.Cu at (152.9, 69.0)
- added R18: R_100K, footprints:R_0805_OEM, F.Cu at (106.2, 63.2)
- added R19: R_22K, footprints:R_0805_OEM, F.Cu at (141.2, 71.1)
- added R20: R_1k, footprints:R_0805_OEM, F.Cu at (119.9, 51.6)
- added R21: R_100k, footprints:R_0805_OEM, F.Cu at (121.9, 51.6)
- added R22: R_10k, footprints:R_0805_OEM, F.Cu at (128.0, 51.4)
- added R23: R_1k, footprints:R_0805_OEM, F.Cu at (112.3, 58.2)
- added R24: R_100k, footprints:R_0805_OEM, F.Cu at (114.3, 58.2)
- added R25: R_10k, footprints:R_0805_OEM, F.Cu at (120.4, 58.2)
- added R26: R_120 DNP, footprints:R_0805_OEM, F.Cu at (135.5, 93.9)
- added R27: R_1k, footprints:R_0805_OEM, F.Cu at (106.4, 49.3)
- added R28: R_100k, footprints:R_0805_OEM, F.Cu at (108.5, 49.3)
- added R29: R_10k, footprints:R_0805_OEM, F.Cu at (114.6, 49.3)
- added R30: R_100, footprints:R_0805_OEM, F.Cu at (127.6, 72.8)
- added R31: R_10k, footprints:R_0805_OEM, F.Cu at (122.2, 64.3)
- added R6: R_1k, footprints:R_0805_OEM, F.Cu at (144.3, 64.8)
- added R7: R_2.2k, footprints:R_0805_OEM, F.Cu at (146.8, 63.5)
- added R8: R_200, footprints:R_0805_OEM, F.Cu at (141.8, 57.9)
- added R_1: R_200, footprints:R_0805_OEM, F.Cu at (131.0, 74.8)
- added R_2: R_200, footprints:R_0805_OEM, F.Cu at (133.8, 74.3)
- added U1: MCP6001, footprints:SOT-23-5_OEM, F.Cu at (143.8, 61.9)
- added U3: MCP6001, footprints:SOT-23-5_OEM, F.Cu at (150.1, 67.6)
- added U4: CAN_Transceiver, footprints:SOIC-8_3.9x4.9mm_Pitch1.27mm_OEM, F.Cu at (135.5, 89.1)
- added Y1: Crystal_SMD, footprints:Crystal_SMD_FA238, F.Cu at (137.3, 74.7)
- C12: value C_0.1uF -> C_47uF
- C7: value C_47uF -> C_0.1uF
- moved U2 30.8 mm to (118.7, 88.6)
- moved C5 30.8 mm to (121.7, 89.9)
- moved L1 30.8 mm to (118.7, 82.0)
- moved R4 30.8 mm to (116.8, 92.2)
- moved C11 30.8 mm to (125.5, 81.3)
- moved C12 30.8 mm to (125.5, 83.6)
- moved C3 30.8 mm to (115.3, 88.9)
- moved C7 30.8 mm to (125.5, 79.2)
- moved D1 30.8 mm to (108.5, 81.5)
- moved R12 30.8 mm to (117.1, 72.4)
- moved R2 30.8 mm to (109.2, 85.1)
- moved R3 30.8 mm to (109.2, 87.1)
- moved R9 30.8 mm to (118.5, 75.6)
- moved D2 30.8 mm to (121.2, 72.4)
- moved D7 30.8 mm to (111.0, 74.9)
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Routing:
- net VCC: track 19.6 -> 201.5 mm, vias 0 -> 13
- net /RESET: track 0.00 -> 106.9 mm, vias 0 -> 12
- net /SCK: track 9.81 -> 100.4 mm, vias 0 -> 10
- net /Throttle2_Left_Sense: track 0.00 -> 89.3 mm, vias 0 -> 12
- net /Throttle1_Right_Sense: track 0.00 -> 78.7 mm, vias 0 -> 11
- net /Drive_Mode_Out: track 0.00 -> 77.0 mm, vias 0 -> 10
- net /MOSI: track 0.00 -> 74.9 mm, vias 0 -> 6
- net /MISO: track 2.75 -> 66.7 mm, vias 0 -> 6
- net /CANH: track 0.00 -> 51.7 mm, vias 0 -> 2
- net /LED2: track 0.00 -> 47.6 mm, vias 0 -> 2
- net /CANL: track 0.00 -> 45.3 mm
- net /LED1: track 0.00 -> 41.1 mm, vias 0 -> 2
- net GND: track 61.2 -> 97.0 mm, vias 15 -> 42
- net /ReadyToDrive_LowDrive: track 0.00 -> 31.5 mm, vias 0 -> 2
- net /SS_BOTS_Out_n: track 0.00 -> 26.8 mm, vias 0 -> 2
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Other:
- board outline added: 59.7 x 53.5 mm
- board text added: "MKIV - Throttle Alex Wenstrup"
