File: Boards/Throttle/throttle2.kicad_pcb (KiCad board)
At the start: 2 copper layers, 59.7 x 53.5 mm, 70 parts, among them IC1 ATMEGA16M1, J1 micromatch_female_TOP_ENTRY_l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, J2 micromatch_female_TOP_ENTRY_l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, J3 CONN_02X03, Q1 SSM3K333R, Q2 SSM3K333R, Q3 SSM3K333R, Q4 SSM3K333R, U1 MCP6001, U2 TPS561201, U3 MCP6001, U4 CAN_Transceiver, Y1 Crystal_SMD

Commit message: Worked on layout, finished a VERY rough REV1
Routing:
- net /Drive_Mode_Out: track 77.0 -> 5.40 mm, vias 10 -> 0
- net /SCK: track 100.4 -> 29.0 mm, vias 10 -> 4
- net /MOSI: track 74.9 -> 35.7 mm, vias 6 -> 1
- net /MISO: track 66.7 -> 29.4 mm, vias 6 -> 1
- net /RXCAN: track 24.8 -> 0.00 mm, vias 6 -> 0
- net /TXCAN: track 23.6 -> 0.00 mm, vias 4 -> 0
- net GND: track 97.0 -> 89.6 mm, vias 42 -> 41
- net Net-(C8-Pad1): track 21.5 -> 19.2 mm
- net Net-(R3-Pad2): track 20.7 -> 18.5 mm
