File: Boards/Dashboard Mk4/dashboard_mk4.kicad_pcb (KiCad board)
At the start: 2 copper layers, 17 parts, among them U2 TPS561201

Commit message: Completed rev3 of layout
Parts:
- added C1: C_0.1uF, footprints:C_0805_OEM, F.Cu at (83.0, 56.2)
- added C10: C_30pF, footprints:C_0805_OEM, F.Cu at (113.5, 53.2)
- added C13: C_30pF, footprints:C_0805_OEM, F.Cu at (85.1, 46.0)
- added C14: C_30pF, footprints:C_0805_OEM, F.Cu at (82.6, 43.1)
- added C15: C_0.1uF, footprints:C_0805_OEM, F.Cu at (75.7, 66.4)
- added C2: C_100pF, footprints:C_0805_OEM, F.Cu at (71.1, 43.3)
- added C4: C_0.1uF, footprints:C_0805_OEM, F.Cu at (110.0, 60.5)
- added C6: C_0.1uF, footprints:C_0805_OEM, F.Cu at (93.2, 63.3)
- added C8: C_0.1uF, footprints:C_0805_OEM, F.Cu at (93.1, 59.1)
- added C9: C_30pF, footprints:C_0805_OEM, F.Cu at (110.3, 56.0)
- added D3: LED, formula:LED_0805_OEM, F.Cu at (104.1, 43.4)
- added D4: LED, formula:LED_0805_OEM, F.Cu at (102.0, 43.4)
- added D5: LED, formula:LED_0805_OEM, F.Cu at (64.6, 56.7)
- added D6: LED, formula:LED_0805_OEM, F.Cu at (66.0, 58.3)
- added D8: LED, formula:LED_0805_OEM, F.Cu at (67.5, 59.8)
- added J1: MM_F_VT_10, footprints:micromatch_female_vert_10, F.Cu at (40.6, 39.8)
- added J2: MM_F_VT_20, footprints:micromatch_female_vert_20, F.Cu at (60.1, 63.1)
- added J3: MM_F_VT_04, footprints:micromatch_female_vert_4, F.Cu at (111.1, 47.4)
- added J4: CONN_02X03, footprints:Pin_Header_Straight_2x03, F.Cu at (93.8, 43.0)
- added J5: CONN_02X03, footprints:Pin_Header_Straight_2x03, F.Cu at (63.8, 34.8)
- added R1: R_200, footprints:R_0805_OEM, F.Cu at (74.5, 59.2)
- added R10: R_200, footprints:R_0805_OEM, F.Cu at (69.1, 45.5)
- added R11: R_200, footprints:R_0805_OEM, F.Cu at (101.9, 47.5)
- added R13: R_200, footprints:R_0805_OEM, F.Cu at (67.6, 47.0)
- added R14: R_200, footprints:R_0805_OEM, F.Cu at (68.2, 53.5)
- added R15: R_200, footprints:R_0805_OEM, F.Cu at (69.7, 55.0)
- added R16: R_200, footprints:R_0805_OEM, F.Cu at (71.2, 56.5)
- added R17: R_100K, footprints:R_0805_OEM, F.Cu at (93.2, 61.2)
- added R18: R_100K, footprints:R_0805_OEM, F.Cu at (93.0, 57.1)
- added R19: R_200, footprints:R_0805_OEM, F.Cu at (66.0, 48.6)
- added R20: R_10K, footprints:R_0805_OEM, F.Cu at (102.6, 66.0)
- added R21: R_10k, footprints:R_0805_OEM, F.Cu at (80.2, 59.5)
- added R22: R_120, footprints:R_0805_OEM, F.Cu at (65.4, 66.4)
- added R6: R_200, footprints:R_0805_OEM, F.Cu at (76.0, 60.6)
- added R7: R_100, footprints:R_0805_OEM, F.Cu at (77.6, 40.0)
- added R8: R_200, footprints:R_0805_OEM, F.Cu at (104.1, 47.5)
- added U1: ATMEGA16M1, footprints:TQFP-32_7x7mm_Pitch0.8mm, F.Cu at (76.1, 50.3)
- added U3: ATmega328P-AU, footprints:TQFP-32_7x7mm_Pitch0.8mm, F.Cu at (101.9, 57.4)
- added U4: CAN_Transceiver, footprints:SOIC-8_3.9x4.9mm_Pitch1.27mm_OEM, F.Cu at (70.5, 66.3)
- added Y1: Crystal_SMD, footprints:Crystal_SMD_FA238, F.Cu at (110.2, 53.3)
- added Y2: Crystal_SMD, footprints:Crystal_SMD_FA238, F.Cu at (85.4, 42.9)
- C12: value C_0.1uF -> C_47uF
- C7: value C_47uF -> C_0.1uF
- moved R5 126.8 mm to (36.1, 51.1), turned to 270 degrees
- moved C12 122.1 mm to (35.6, 57.7), turned to 180 degrees
- moved C5 120.8 mm to (39.4, 51.3), turned to 270 degrees
- moved C11 120.5 mm to (35.6, 59.9), turned to 180 degrees
- moved C7 119.1 mm to (35.6, 62.0), turned to 180 degrees
- moved R4 114.9 mm to (44.2, 49.0), turned to 0 degrees
- moved U2 114.2 mm to (42.4, 52.6), turned to 90 degrees
- moved C3 108.8 mm to (45.7, 52.3), turned to 90 degrees
- moved L1 108.4 mm to (42.3, 59.2), turned to 270 degrees
- moved D2 107.1 mm to (39.9, 68.8), turned to 0 degrees
- moved R9 103.6 mm to (42.5, 65.7), turned to 180 degrees
- moved R12 99.2 mm to (43.9, 68.8), turned to 180 degrees
- moved F1 97.6 mm to (48.7, 58.5), turned to 90 degrees
- moved R3 96.6 mm to (51.8, 54.1), turned to 0 degrees
- moved R2 94.4 mm to (51.8, 56.1), turned to 0 degrees
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Routing:
- net VCC: track 19.6 -> 200.3 mm
- net /RESET: track 0.00 -> 61.5 mm
- net /MOSI: track 0.00 -> 56.5 mm, vias 0 -> 2
- net /MISO: track 2.75 -> 55.4 mm, vias 0 -> 2
- net /TXCAN: track 0.00 -> 45.9 mm, vias 0 -> 4
- net /SCL: track 0.00 -> 44.4 mm, vias 0 -> 2
- net /SCK: track 9.81 -> 52.9 mm, vias 0 -> 2
- net /STR_POT_SENSE: track 0.00 -> 43.0 mm, vias 0 -> 2
- net /SDA: track 0.00 -> 36.0 mm, vias 0 -> 4
- net /PWM_0: track 0.00 -> 34.6 mm, vias 0 -> 6
- net Net-(R1-Pad2): track 0.00 -> 31.9 mm, vias 0 -> 4
- net /RESET_2: track 0.00 -> 29.3 mm, vias 0 -> 2
- net /RXCAN: track 4.11 -> 33.4 mm, vias 0 -> 4
- net Net-(R6-Pad2): track 0.00 -> 24.5 mm, vias 0 -> 4
- net GND: track 61.2 -> 85.3 mm, vias 15 -> 40
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Other:
- board outline added: 87.9 x 50.6 mm
- board text added: "Aditya Sudhakar Dashboard - Right - v3 Olin Electric Motorsports MKIV"
- board text added: "CAN Bus"
- board text added: "DNP"
- board text added: "Debugging"
- board text added: "MISO2|VCC SCK2|MOSI2 RST2|GND"
- board text added: "MISO|VCC SCK|MOSI RST|GND"
- board text added: "Structural Support"
