File: Boards/Steering/Steering.kicad_pcb (KiCad board)
At the start: 2 copper layers, 76.2 x 21.3 mm, 44 parts, among them IC1 ATMEGA16M1, J1 MM_F_VT_14, J2 MM_F_VT_04, J4 CONN_02X03, U1 MCP2561-E_SN, U2 TPS561201, Y1 Crystal_SMD

Commit message: Updating Labels, C1 and Y1 placements
Parts:
- moved C1 17.4 mm to (146.5, 67.3), turned to 180 degrees
- moved C2 3.83 mm to (157.5, 79.2), turned to 0 degrees
- moved D4 1.52 mm to (177.5, 79.0)
- moved D5 1.52 mm to (177.5, 83.3)
- moved D6 1.52 mm to (177.5, 81.0)
- moved C8 1.48 mm to (143.3, 78.0)
- moved Y1 1.37 mm to (146.0, 77.3)
- moved C6 1.37 mm to (146.0, 80.5)
- moved R1 0.77 mm to (157.5, 77.2), turned to 180 degrees
Routing:
- net Net-(C2-Pad1): track 7.68 -> 5.29 mm
- net VCC: track 121.7 -> 120.1 mm
- net Net-(D6-Pad2): track 2.44 -> 3.96 mm
- net Net-(D5-Pad2): track 2.44 -> 3.96 mm
- net Net-(D4-Pad2): track 2.44 -> 3.96 mm
- net Net-(C6-Pad1): track 7.90 -> 6.67 mm
- net GND: track 74.7 -> 75.8 mm, vias 13 -> 14
- net Net-(C8-Pad1): track 7.45 -> 6.74 mm
- net /RESET: track 19.3 -> 19.8 mm
Other:
- rule trace_min: 0.2 -> 0.1778
- board text added: "PB2"
- board text added: "PD6"
- board text added: "PD7"
- board text added: "Things to figure out: mounting holes (is what they're referred to as) are placed on there by mechanical in their DXF -placement looks not-too-concerning on J2,U2 -I would not recommend using micrmatch to interface with the buttons or LEDs. Micromatches are used to interface a lot of wires between board to board or board to wire. While possible, it'd be unnecessarily inconvenient and just bad (alt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"
- board text removed: "Things to figure out: - Screw Holes - how to actually connect to board - Are any pieces to close (J2,U2) - Other labels - how micromatch works specifically for the button and led ins and outs"
