File: Boards/Steering/REV1/Steering.kicad_pcb (KiCad board)
At the start: 2 copper layers, 76.2 x 21.3 mm, 44 parts, among them IC1 ATMEGA16M1, J1 MM_F_VT_14, J2 MM_F_VT_04, J4 CONN_02X03, U1 MCP2561-E_SN, U2 TPS561201, Y1 Crystal_SMD

Commit message: Redesign of layout to include new nanofit connectors
Parts:
- moved C1 17.4 mm to (146.5, 67.3), turned to 180 degrees
- moved C12 11.5 mm to (122.1, 83.5), turned to 90 degrees
- moved C3 9.80 mm to (122.2, 74.9), turned to 180 degrees
- moved C11 7.98 mm to (124.7, 83.4), turned to 90 degrees
- moved C7 4.61 mm to (127.2, 83.4), turned to 90 degrees
- moved C2 3.83 mm to (157.5, 79.2), turned to 0 degrees
- moved R19 3.78 mm to (130.8, 81.1)
- moved C5 3.36 mm to (119.6, 80.0), turned to 270 degrees
- moved F1 2.36 mm to (120.7, 70.4)
- moved D7 1.87 mm to (120.4, 66.5)
- moved D4 1.52 mm to (177.5, 79.0)
- moved D5 1.52 mm to (177.5, 83.3)
- moved D6 1.52 mm to (177.5, 81.0)
- moved C8 1.48 mm to (143.3, 78.0)
- moved Y1 1.37 mm to (146.0, 77.3)
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Routing:
- net Net-(R18-Pad1): track 6.07 -> 20.8 mm, vias 0 -> 2
- net /12V_Fused: track 24.5 -> 16.8 mm
- net +12V: track 11.7 -> 5.55 mm
- net Net-(C5-Pad1): track 7.37 -> 2.15 mm, vias 2 -> 0
- net Net-(C11-Pad1): track 22.7 -> 18.2 mm
- net GND: track 74.7 -> 78.0 mm, vias 13 -> 12
- net Net-(R17-Pad1): track 10.7 -> 7.84 mm
- net Net-(C2-Pad1): track 7.68 -> 5.29 mm
- net Net-(C5-Pad2): track 15.2 -> 17.0 mm, vias 0 -> 2
- net VCC: track 121.7 -> 120.1 mm
- net Net-(D6-Pad2): track 2.44 -> 3.96 mm
- net Net-(D5-Pad2): track 2.44 -> 3.96 mm
- net Net-(D4-Pad2): track 2.44 -> 3.96 mm
- net Net-(C6-Pad1): track 7.90 -> 6.67 mm
- net Net-(C8-Pad1): track 7.45 -> 6.74 mm
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- added copper zone on F.Cu, net GND
Other:
- net class Default: clearance 0.1524 -> 0.2; trace_width 0.1524 -> 0.25
- board text added: "PB2"
- board text added: "PD6"
- board text added: "PD7"
- board text added: "Things to figure out: mounting holes (is what they're referred to as) are placed on there by mechanical in their DXF -I would not recommend using micrmatch to interface with the buttons or LEDs. Micromatches are used to interface a lot of wires between board to board or board to wire. While possible, it'd be unnecessarily inconvenient and just bad (although you didn't know that) -If possible, I'd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"
- board text removed: "Things to figure out: - Screw Holes - how to actually connect to board - Are any pieces to close (J2,U2) - Other labels - how micromatch works specifically for the button and led ins and outs"
