File: Boards/MKIV_IMU/IMU.kicad_pcb (KiCad board)
At the start: 2 copper layers, 50.8 x 55.9 mm, 42 parts, among them J1 UF_4_VT, J4 CONN_02X03, U1 CAN_Transceiver, U2 TPS561201, U3 LM3480, U4 BMI088, U5 ATMEGA16M1, Y1 Crystal_SMD

Commit message: layout stuffffffffffff
Parts:
- moved R7 27.6 mm to (126.1, 100.4)
- moved C8 27.4 mm to (149.9, 100.8), turned to 270 degrees
- moved J4 26.7 mm to (125.1, 87.3), turned to 270 degrees
- moved U1 26.4 mm to (130.8, 100.4)
- moved Y1 22.3 mm to (151.0, 97.4)
- moved C6 22.2 mm to (152.1, 94.0)
- moved R11 15.3 mm to (129.2, 91.2), turned to 180 degrees
- moved R6 14.5 mm to (129.2, 86.1), turned to 180 degrees
- moved R10 14.4 mm to (129.2, 88.6), turned to 180 degrees
- moved D1 13.6 mm to (127.8, 114.4)
- moved C5 13.4 mm to (140.9, 122.2)
- moved R12 13.4 mm to (136.3, 104.7)
- moved C3 13.4 mm to (134.6, 121.2)
- moved D7 13.4 mm to (130.2, 107.2)
- moved C11 13.4 mm to (144.7, 113.5)
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Connections:
- U5 pad 10: Net-(U5-Pad10) -> Net-(C8-Pad1)
Routing:
- net VCC: track 97.6 -> 7.72 mm, vias 2 -> 0
- net GND: track 80.3 -> 28.0 mm, vias 23 -> 14
- net /SCK: track 35.4 -> 0.00 mm, vias 1 -> 0
- net /INT4: track 34.4 -> 0.00 mm, vias 2 -> 0
- net /CANH: track 33.5 -> 0.00 mm
- net /CANL: track 33.0 -> 0.00 mm
- net /CS_GYRO: track 32.5 -> 0.00 mm, vias 2 -> 0
- net /12V: track 27.6 -> 4.95 mm
- net /INT2: track 22.9 -> 5.70 mm, vias 2 -> 0
- net /INT1: track 19.4 -> 3.47 mm, vias 2 -> 0
- net /CS_ACCEL: track 13.3 -> 0.00 mm, vias 2 -> 0
- net /RESET: track 14.9 -> 2.01 mm, vias 1 -> 0
- net /INT3: track 12.8 -> 0.00 mm, vias 2 -> 0
- net /TXCAN: track 9.30 -> 21.9 mm, vias 2 -> 0
- net /SCK2: track 12.5 -> 0.00 mm, vias 2 -> 0
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Other:
- rule trace_min: 0.2 -> 0.1524

Commit message: layout progress
Parts:
- moved R1 15.6 mm to (157.8, 90.2), turned to 225 degrees
- moved C10 10.4 mm to (158.4, 74.4)
- moved J1 10.3 mm to (122.4, 109.6)
- moved C9 9.36 mm to (161.5, 77.3), turned to 90 degrees
- moved J4 8.38 mm to (132.3, 91.5)
- moved R6 8.36 mm to (135.8, 81.0), turned to 135 degrees
- moved R11 8.31 mm to (132.9, 83.8), turned to 135 degrees
- moved R10 8.12 mm to (134.3, 82.4), turned to 135 degrees
- moved C14 7.69 mm to (155.6, 77.6), turned to 90 degrees
- moved U3 7.35 mm to (157.4, 77.3), turned to 0 degrees
- moved C6 7.06 mm to (152.2, 101.0), turned to 270 degrees
- moved C1 6.26 mm to (136.1, 96.7), turned to 135 degrees
- moved D3 5.92 mm to (138.3, 83.6), turned to 315 degrees
- moved D5 5.47 mm to (135.5, 86.3), turned to 315 degrees
- moved D4 5.39 mm to (136.9, 84.9), turned to 315 degrees
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Connections:
- C10 pad 2: Net-(C10-Pad2) -> GND
- C9 pad 2: Net-(C10-Pad2) -> GND
Routing:
- net /RESET: track 2.01 -> 12.8 mm
- net /MOSI: track 0.00 -> 10.5 mm
- net /CANH: track 0.00 -> 10.2 mm
- net /INT3: track 0.00 -> 8.94 mm
- net /INT4: track 0.00 -> 8.74 mm
- net /12V: track 4.95 -> 13.7 mm
- net /CANL: track 0.00 -> 8.61 mm
- net /RXCAN: track 16.2 -> 8.10 mm
- net /TXCAN: track 21.9 -> 14.5 mm
- net Net-(C6-Pad1): track 6.97 -> 0.00 mm
- net /MISO: track 0.00 -> 6.89 mm
- net /PLED1: track 0.00 -> 5.89 mm
- net /INT2: track 5.70 -> 0.00 mm
- net /PLED3: track 0.00 -> 5.56 mm
- net /PLED2: track 0.00 -> 5.45 mm
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
Commit message: more layout stuff
Parts:
- moved C14 12.4 mm to (143.4, 79.5)
- moved U3 12.3 mm to (145.2, 79.0)
- moved C10 12.3 mm to (146.2, 76.1)
- moved C9 12.3 mm to (149.3, 79.0)
- moved R1 10.3 mm to (147.7, 88.1)
- moved U4 7.26 mm to (143.8, 82.8), turned to 0 degrees
- moved C13 2.65 mm to (145.9, 85.3), turned to 180 degrees
- moved C2 1.36 mm to (148.5, 90.0), turned to 45 degrees
Routing:
- net VCC: track 8.84 -> 83.0 mm, vias 0 -> 3
- net GND: track 26.6 -> 65.9 mm, vias 11 -> 26
- net /INT1: track 0.00 -> 33.2 mm
- net /INT2: track 0.00 -> 30.4 mm
- net /SCK: track 0.00 -> 22.5 mm, vias 0 -> 1
- net /CS_ACCEL: track 0.00 -> 13.2 mm
- net /SCK2: track 0.00 -> 12.8 mm, vias 0 -> 2
- net /CS_GYRO: track 0.00 -> 12.7 mm, vias 0 -> 2
- net /3.3V: track 1.70 -> 11.2 mm
- net Net-(C6-Pad1): track 0.00 -> 8.47 mm
- net Net-(C8-Pad1): track 0.00 -> 6.12 mm
- net /INT4: track 8.74 -> 5.29 mm
- net Net-(D2-Pad2): track 0.00 -> 2.35 mm
- net Net-(C2-Pad1): track 2.08 -> 4.09 mm
- net Net-(D1-Pad2): track 0.00 -> 1.97 mm
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
Commit message: even more layout changesgit add IMU.kicad_pcb-bak
Parts:
- moved C14 6.17 mm to (149.1, 77.1)
- moved C10 6.11 mm to (151.9, 73.9)
- moved U3 6.11 mm to (150.9, 76.8)
- moved C9 6.11 mm to (155.0, 76.8)
- moved C11 5.79 mm to (150.4, 112.5)
- moved C12 5.79 mm to (150.4, 114.8)
- moved C6 5.79 mm to (157.9, 100.0)
- moved C7 5.79 mm to (150.4, 110.5)
- moved D5 5.79 mm to (141.2, 85.3)
- moved R10 5.79 mm to (140.0, 81.4)
- moved R12 5.79 mm to (142.0, 103.7)
- moved R2 5.79 mm to (134.2, 116.4)
- moved U5 5.79 mm to (148.4, 93.2)
- moved C1 5.79 mm to (141.8, 95.7)
- moved C5 5.79 mm to (146.6, 121.2)
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Routing:
- net VCC: track 83.0 -> 2.06 mm, vias 3 -> 0
- net /INT1: track 33.2 -> 0.00 mm
- net /INT2: track 30.4 -> 0.00 mm
- net /CANL: track 8.61 -> 14.0 mm
- net /CANH: track 10.2 -> 15.0 mm
- net /MISO2: track 4.02 -> 0.00 mm, vias 2 -> 0
- net /3.3V: track 11.2 -> 13.1 mm
- net GND: track 65.9 -> 66.7 mm
