File: Boards/BMS_Structural/_autosave-BMS_Structural.kicad_pcb (KiCad board)
At the start: 2 copper layers, 400.6 x 70.3 mm, 48 parts, among them J1 MM_F_VT_16, J2 MM_F_VT_20, J3 MM_F_VT_20, J4 MM_F_VT_20, Q101 LMT85-Q1, Q102 LMT85-Q1, Q11 LMT85-Q1, Q12 LMT85-Q1, Q21 LMT85-Q1, Q22 LMT85-Q1, Q31 LMT85-Q1, Q32 LMT85-Q1, Q41 LMT85-Q1, Q42 LMT85-Q1, Q51 LMT85-Q1, Q52 LMT85-Q1, Q61 LMT85-Q1, Q62 LMT85-Q1, Q71 LMT85-Q1, Q72 LMT85-Q1, Q81 LMT85-Q1, Q82 LMT85-Q1, Q91 LMT85-Q1, Q92 LMT85-Q1

Commit message: Pushing again
Parts:
- J2: moved to F.Cu
- J4: moved to B.Cu
- moved B8 116.1 mm to (6.23, 107.1)
- moved J2 1.67 mm to (168.3, 90.0), turned to 90 degrees
- moved J4 0.54 mm to (167.6, 74.5), turned to 270 degrees
Routing:
- net /volt9: track 208.7 -> 190.1 mm
- net /volt6: track 207.0 -> 188.4 mm
- net /volt7: track 111.2 -> 92.7 mm
- net /V11: track 244.3 -> 225.8 mm
- net /MODULE8_TEMP2: track 149.2 -> 130.6 mm
- net /MODULE8_TEMP1: track 138.9 -> 120.3 mm
- net /MODULE7_TEMP1: track 171.5 -> 153.0 mm
- net /5V: track 1466.0 -> 1449.7 mm
- net /volt10: track 281.3 -> 265.6 mm
- net /V+: track 296.8 -> 283.1 mm
- net /volt8: track 126.6 -> 113.1 mm
- net /MODULE9_TEMP2: track 231.3 -> 217.8 mm
- net /MODULE9_TEMP1: track 197.5 -> 184.0 mm
- net /MODULE6_TEMP1: track 264.4 -> 250.9 mm
- net /MODULE10_TEMP2: track 296.9 -> 283.4 mm
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