File: Boards/Brakelight_Shutdown_BSPD/rev_1_2-10-19/_autosave-Brakelight_Shutdown_BSPD.kicad_pcb (KiCad board)
At the start: 2 copper layers, 85.1 x 82.6 mm, 91 parts, among them IC1 ATMEGA16M1, J1 MM_F_RA_06, J2 MM_F_RA_20, J3 CONN_02X03, Q1 SSM3K333R, Q2 SSM3K333R, Q3 SSM3K333R, Q4 SSM3K333R, Q5 SSM3K333R, Q6 SSM3K333R, Q7 SSM3K333R, U1 SN74LVC1G08, U2 MCP6001, U3 CAN_Transceiver, U4 TPS561201, U5 SN74LVC1G02, U6 SN74LVC1G02, U7 MCP6001, Y1 Crystal_SMD

Commit message: Created folder for first revision board and started updated version
Parts:
- removed D11: LED_0805, footprints:LED_0805_OEM
- removed R36: R_1K-formula, footprints:R_0805_OEM
- moved R16 80.4 mm to (239.5, 101.1), turned to 90 degrees
- moved C12 79.6 mm to (240.0, 94.5), turned to 0 degrees
- moved C13 79.4 mm to (240.0, 92.2), turned to 0 degrees
- moved C14 79.3 mm to (240.0, 90.2), turned to 0 degrees
- moved C11 75.7 mm to (236.2, 100.8), turned to 90 degrees
- moved D6 73.6 mm to (235.7, 83.3), turned to 180 degrees
- moved R34 71.3 mm to (181.9, 48.8), turned to 180 degrees
- moved J3 71.3 mm to (169.4, 38.0)
- moved U4 71.2 mm to (233.2, 99.5), turned to 270 degrees
- moved R15 69.9 mm to (231.4, 103.1), turned to 180 degrees
- moved L1 69.9 mm to (233.2, 92.9), turned to 90 degrees
- moved R19 69.5 mm to (233.0, 86.5), turned to 0 degrees
- moved R2 68.2 mm to (198.8, 39.3), turned to 180 degrees
- moved R20 67.9 mm to (231.6, 83.3), turned to 0 degrees
- moved C7 66.6 mm to (229.9, 99.8), turned to 270 degrees
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Connections:
- IC1 pad 30: /Cooling_Pump_LSD -> /Cooling_Pump_LSD_n
- J2 pad 13: /Cooling_Pump_LSD -> /Cooling_Pump_LSD_n
Routing:
- net VCC: track 53.1 -> 304.4 mm, vias 0 -> 18
- net +12V: track 22.4 -> 154.7 mm, vias 0 -> 1
- net /BSPD_Current_Sense: track 25.1 -> 151.1 mm, vias 0 -> 4
- net /BSPD_Relay_Sense: track 0.00 -> 95.6 mm
- net GND: track 29.1 -> 109.6 mm, vias 14 -> 58
- net /SCK: track 7.80 -> 74.3 mm, vias 0 -> 5
- net /BSPD_Relay: track 9.46 -> 72.3 mm, vias 0 -> 4
- net /MISO: track 9.14 -> 70.3 mm, vias 0 -> 4
- net /MOSI: track 9.08 -> 69.0 mm, vias 0 -> 4
- net /Shutdown_Sense_Estop: track 0.00 -> 58.9 mm, vias 0 -> 2
- net /Brake_Pressure_Sense: track 0.00 -> 51.5 mm
- net /Shutdown_Sense_TSMS: track 0.00 -> 51.4 mm, vias 0 -> 2
- net /RESET: track 27.6 -> 78.2 mm, vias 0 -> 5
- net /Brake_Pressure-: track 0.00 -> 50.2 mm
- net /Brakelight_Gate: track 0.00 -> 50.0 mm
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