File: Boards/Interface_DashLeft/interface/interface.kicad_pcb (KiCad board)
At the start: 2 copper layers, 6 parts, among them J1 UF_2_VT, J2 MM_F_VT_08, J3 Ampseal_23_VT, J4 MM_F_VT_04, J5 MM_F_VT_20, U1 RJ45_VT

Commit message: Finished Rev1 DashLeft Interface Layout
Parts:
- added G***: LOGO, footprints:Logo_Large, F.Cu at (87.8, 97.9)
- J1, J2, J3, U1: moved to B.Cu
- J4, J5: moved to F.Cu
- moved J1 206.8 mm to (18.2, 81.5)
- moved J2 155.1 mm to (63.5, 114.5), turned to 90 degrees
- moved U1 135.1 mm to (25.8, 113.9), turned to 90 degrees
- moved J4 127.1 mm to (85.2, 71.4), turned to 270 degrees
- moved J5 126.9 mm to (60.6, 105.0), turned to 270 degrees
- moved J3 110.6 mm to (69.9, 88.7), turned to 180 degrees
Connections:
- J4 pad 1: /SS_BOTS -> /BOTS->ESTOP
- J4 pad 2: /SS_IS -> /IS->BOTS
- J4 pad 3: /SS_ESTOP -> /ESTOP->HVD
Routing:
- net /ESTOP->HVD: track 0.00 -> 87.2 mm
- net /BOTS->ESTOP: track 0.00 -> 80.4 mm, vias 0 -> 2
- net /IS->BOTS: track 0.00 -> 63.4 mm, vias 0 -> 2
- net /MOSI: track 0.00 -> 51.2 mm
- net /CANH: track 0.00 -> 44.5 mm
- net /SCK: track 0.00 -> 44.3 mm
- net /CANL: track 0.00 -> 44.2 mm
- net /MISO: track 0.00 -> 42.5 mm
- net /SDA: track 0.00 -> 40.6 mm, vias 0 -> 2
- net /12V: track 0.00 -> 39.6 mm
- net /RTD_LSD_GND: track 0.00 -> 39.4 mm, vias 0 -> 2
- net /SCL: track 0.00 -> 37.5 mm, vias 0 -> 2
- net /LED2: track 0.00 -> 31.1 mm
- net /RESET: track 0.00 -> 28.7 mm
- net /LED1: track 0.00 -> 19.8 mm
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- added copper zone on B.Cu, net /GND
Other:
- board outline added: 83.8 x 53.3 mm
- net class Default: trace_width 0.25 -> 0.1524
- net class Power added: clearance 0.2, trace_width 0.254, via_dia 0.8, via_drill 0.4
- net class Shutdown added: clearance 0.2, trace_width 0.762, via_dia 0.8, via_drill 0.4
- rule trace_min: 0.2 -> 0.1524
- board text added: "Dashboard Left Interface Board Alex Wenstrup"
- board text removed: "For Instructional Use Only."
- board text removed: "SOLIDWORKS Educational Product."

Commit message: Updated Interface
Parts:
- J2: moved to F.Cu
- moved J1 68.6 mm to (86.7, 82.2), turned to 180 degrees
- moved G*** 60.7 mm to (32.4, 73.3), turned to 0 degrees
- moved U1 8.37 mm to (19.7, 108.2), turned to 0 degrees
- moved J2 2.61 mm to (66.0, 115.3), turned to 270 degrees
- moved J3 1.00 mm to (69.4, 87.9)
- moved J4 1.00 mm to (84.6, 70.5)
Routing:
- net /ESTOP->HVD: track 87.2 -> 62.7 mm, vias 0 -> 2
- net /CANH: track 44.5 -> 65.0 mm
- net /BOTS->ESTOP: track 80.4 -> 62.8 mm, vias 2 -> 0
- net /Drive_Select-: track 8.42 -> 22.2 mm, vias 0 -> 2
- net /MOSI: track 51.2 -> 37.4 mm
- net /CANL: track 44.2 -> 56.8 mm
- net /MISO: track 42.5 -> 33.8 mm, vias 0 -> 2
- net /Drive_Select+: track 7.08 -> 15.3 mm
- net /LED2: track 31.1 -> 23.0 mm
- net /SCK: track 44.3 -> 36.6 mm
- net /Drive_Select_Sense: track 4.77 -> 12.5 mm
- net /LED1: track 19.8 -> 13.9 mm
- net /RESET: track 28.7 -> 33.6 mm
- net /SDA: track 40.6 -> 44.8 mm
- net /SCL: track 37.5 -> 41.3 mm
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
Commit message: Rev1 dashleft layout gerbers
Parts:
- J1: moved to F.Cu
- moved J2 5.44 mm to (62.9, 119.8)
- moved G*** 1.98 mm to (34.4, 73.5)
- moved J4 0.96 mm to (85.2, 71.3)
- moved J1 0.09 mm to (86.8, 82.3), turned to 0 degrees
Routing:
- net /Drive_Select-: track 22.2 -> 28.8 mm
- net /Drive_Select_Sense: track 12.5 -> 18.6 mm
- net /5V: track 9.59 -> 15.4 mm
- net /Drive_Select+: track 15.3 -> 21.1 mm
- net /SCL: track 41.3 -> 40.1 mm
- net /SDA: track 44.8 -> 43.6 mm
- net /ESTOP->HVD: track 62.7 -> 63.7 mm
- net /IS->BOTS: track 64.8 -> 65.8 mm
- net /BOTS->ESTOP: track 62.8 -> 62.2 mm
Other:
- board size 83.8 x 53.3 mm -> 83.8 x 61 mm

Commit message: Updated both rev4 throttle and rev2 interface
Parts:
- moved J1 68.3 mm to (19.0, 74.1), turned to 180 degrees
- moved G*** 65.8 mm to (91.9, 105.5), turned to 270 degrees
Routing:
- net /BOTS->ESTOP: track 62.2 -> 86.0 mm, vias 0 -> 2
- net /ESTOP->HVD: track 63.7 -> 85.2 mm, vias 2 -> 0
- net /IS->BOTS: track 65.8 -> 67.0 mm, vias 0 -> 2
