File: Boards/Throttle/REV4/throttle.kicad_pcb (KiCad board)
At the start: 2 copper layers, 203.6 x 151.8 mm, 71 parts, among them IC1 ATMEGA16M1, J1 micromatch_female_TOP_ENTRY_l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, J2 micromatch_female_TOP_ENTRY_l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, J3 CONN_02X03, Q1 SSM3K333R, Q2 SSM3K333R, Q3 SSM3K333R, Q4 SSM3K333R, U1 MCP6001, U2 TPS561201, U3 MCP6001, U4 CAN_Transceiver, Y1 Crystal_SMD

Commit message: Updated both rev4 throttle and rev2 interface
Parts:
- removed the PB4 at (248.7, 56.0)
- removed the PB4 at (248.8, 52.7)
- added PB3: LED_0805, footprints:LED_0805_OEM, F.Cu at (86.8, 120.0)
- added PB4: LED_0805, footprints:LED_0805_OEM, F.Cu at (87.1, 116.7)
- moved R15 180.5 mm to (66.3, 154.8), turned to 357 degrees
- moved R19 177.7 mm to (72.7, 155.2), turned to 357 degrees
- moved R5 175.8 mm to (97.9, 154.0), turned to 87 degrees
- moved R4 175.8 mm to (89.6, 155.6), turned to 177 degrees
- moved C5 175.8 mm to (94.6, 153.6), turned to 87 degrees
- moved U2 175.6 mm to (91.7, 152.1), turned to 267 degrees
- moved C3 175.6 mm to (88.3, 152.3), turned to 267 degrees
- moved C12 175.5 mm to (98.7, 147.5), turned to 357 degrees
- moved C11 175.4 mm to (98.8, 145.2), turned to 357 degrees
- moved R3 175.4 mm to (82.3, 150.2), turned to 177 degrees
- moved C7 175.3 mm to (99.0, 143.2), turned to 357 degrees
- moved L1 175.3 mm to (92.0, 145.5), turned to 87 degrees
- moved R2 175.3 mm to (82.4, 148.1), turned to 177 degrees
- moved F1 175.2 mm to (85.7, 145.9), turned to 267 degrees
- moved D1 175.1 mm to (81.8, 144.5), turned to 267 degrees
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Connections:
- IC1 pad 25: Net-(IC1-Pad25) -> /ReadyToDrive_LowDrive
- J1 pad 4: GND -> /RTD
Routing:
- net /SS_BOTS: track 36.3 -> 58.0 mm
- net /SS_Inertia_Switch: track 33.4 -> 44.2 mm
- net /SS_BOTS_Out_n: track 6.62 -> 15.0 mm
- net Net-(IC1-Pad25): track 7.12 -> 0.00 mm, vias 1 -> 0
- net /ReadyToDrive_LowDrive: track 14.2 -> 21.3 mm, vias 1 -> 2
- net VCC: track 179.3 -> 184.9 mm, vias 6 -> 8
- net /SS_Inertia_Out_n: track 7.27 -> 12.6 mm
- net /Throttle1_Right_Sense: track 47.8 -> 52.3 mm, vias 6 -> 8
- net Net-(IC1-Pad9): track 32.4 -> 28.2 mm
- net +12V: track 24.9 -> 21.4 mm
- net /LED1: track 5.44 -> 1.96 mm
- net /Drive_Mode_Out: track 25.3 -> 28.2 mm
- net /MOSI: track 28.3 -> 25.8 mm
- net /SCK: track 30.3 -> 27.9 mm
- net /CANH: track 11.3 -> 8.92 mm
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Other:
- board size 203.6 x 151.8 mm -> 92.9 x 62.1 mm
- board text added: "DMO"
- board text added: "T-LS"
- board text added: "T-RS"
- board text removed: "For Instructional Use Only."
- board text removed: "SOLIDWORKS Educational Product."
