File: Boards/Sensing_Module/sensing_board.kicad_pcb (KiCad board)
At the start: 2 copper layers, 44.5 x 87.4 mm, 45 parts, among them IC1 ATMEGA16M1, J1 Ampseal_35_RA, U1 CAN_Transceiver, U2 TPS560430YF, U3 LMV341, U7 SK812, U8 USB_MicroB, Y1 Crystal_SMD

Commit message: updated air ctrl board and sensing board
Parts:
- moved C2 16.6 mm to (207.8, 97.9), turned to 270 degrees
- moved G*** 0.90 mm to (208.3, 94.6)
Connections:
- IC1 pad 14: Net-(IC1-Pad14) -> /BRAKETEMP
- IC1 pad 15: Net-(IC1-Pad15) -> /HSENSOR
- IC1 pad 26: /BRAKETEMP -> Net-(IC1-Pad26)
- IC1 pad 27: /HSENSOR -> Net-(IC1-Pad27)
- J1 pad 10: VCC -> Net-(J1-Pad10)
- J1 pad 11: /BRAKETEMP -> Net-(J1-Pad11)
- J1 pad 14: /HSENSOR -> GND
- J1 pad 16: VCC -> /CANL
- J1 pad 17: /POT -> /CANH
- J1 pad 18: GND -> VCC
- J1 pad 19: GND -> VCC
- J1 pad 2: GND -> /12V
- J1 pad 30: Net-(J1-Pad30) -> GND
- J1 pad 31: Net-(J1-Pad31) -> GND
- J1 pad 32: Net-(J1-Pad32) -> GND
- J1 pad 33: Net-(J1-Pad33) -> GND
- J1 pad 34: Net-(J1-Pad34) -> GND
- J1 pad 35: Net-(J1-Pad35) -> GND
- J1 pad 4: /12V -> /CANL
- J1 pad 5: /CANL -> /CANH
- J1 pad 6: /CANH -> /BRAKETEMP
- J1 pad 7: /CANL -> /HSENSOR
- J1 pad 8: /CANH -> /POT
- J1 pad 9: GND -> Net-(J1-Pad9)
Routing:
- net /BRAKETEMP: track 37.3 -> 14.9 mm
- net /HSENSOR: track 33.5 -> 16.2 mm, vias 5 -> 0
- net /CANL: track 27.9 -> 19.2 mm
- net /CANH: track 30.0 -> 21.9 mm
- net /POT: track 16.6 -> 11.8 mm, vias 1 -> 0
- net /12V: track 32.3 -> 34.4 mm, vias 0 -> 2
- net VCC: track 240.3 -> 238.7 mm, vias 8 -> 6
- net /P_LED_1: track 40.5 -> 38.9 mm, vias 6 -> 4
- net GND: track 77.2 -> 75.8 mm, vias 24 -> 26
- net /MISO: track 37.2 -> 38.5 mm, vias 4 -> 2
- net /NEO_PIXEL: track 42.3 -> 42.7 mm, vias 2 -> 0
- net /RESET: track 45.9 -> 46.3 mm, vias 6 -> 4
- net Net-(D4-Pad2): track 5.66 -> 5.94 mm, vias 0 -> 2
- net /MOSI: track 38.0 -> 37.7 mm, vias 4 -> 2
